File: pcb/right-part.kicad_sch (KiCad schematic)
At the start: 67 parts, among them J6 MJ-4PP-9, SW24 SW_PUSH, SW25 SW_PUSH, SW26 SW_PUSH, SW27 SW_PUSH, SW28 SW_PUSH, SW29 SW_PUSH, SW30 SW_PUSH, SW31 SW_PUSH, SW32 SW_PUSH, SW33 SW_PUSH, SW34 SW_PUSH, SW35 SW_PUSH, SW36 SW_PUSH, SW37 SW_PUSH, SW38 SW_PUSH, SW39 SW_PUSH, SW40 SW_PUSH, SW41 SW_PUSH, SW42 SW_RESET, SW43 SW_PUSH, SW44 SW_PUSH, SW45 SW_PUSH, SW46 SW_PUSH, SW53 SW_PUSH, SW54 SW_PUSH, SW55 SW_PUSH, SW56 SW_PUSH, SW57 SW_PUSH, SW58 SW_PUSH, U2 Raspberry_Pie_Pico

Commit message: fixed schematic ERC errors and warnings refactored some symbols to project-level libraries
Parts:
- D23, D24, D25, D26, D27, D28, D29, D30, D31, D32, D33, D34, D35, D36, D37, D38, D39, D40, D41, D42, D43, D44, D63, D64, D65, D66, D67, D68: footprint Keebio-Parts:Diode-Hybrid-Back -> _keebio-parts:Diode-Hybrid-Back
- D53, D54, D55, D56, D57, D59: footprint Yoichiro:LED_WS2812B -> _yoichiro:LED_WS2812B
- J6: footprint kbd:MJ-4PP-9_1side -> _kbd:MJ-4PP-9; symbol kbd:MJ-4PP-9 -> _kbd:MJ-4PP-9
- LS2: footprint Yoichiro:SPKR_PKLCS1212E4001-R1 -> _speaker:SPKR_PKLCS1212E4001-R1; symbol PKLCS1212E4001-R1:PKLCS1212E4001-R1 -> _speaker:PKLCS1212E4001-R1; Availability (none) -> In Stock; Check_prices (none) -> https://www.snapeda.com/parts/PKLCS1212E4001-R1/Murata/view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; Description_1 (none) -> Buzzers Transducer, Externally Driven Piezo 1.5 V - 4kHz 84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; MANUFACTURER (none) -> Murata Electronics; MAXIMUM_PACKAGE_HEIGHT (none) -> 3.0 mm; MF (none) -> Murata; MP (none) -> PKLCS1212E4001-R1; PARTREV (none) -> January 22, 2018; Package (none) -> SMD-2 Murata; Price (none) -> None; Purchase-URL (none) -> https://www.snapeda.com/api/url_track_click_mouser/?unipart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; STANDARD (none) -> Manufacturer Recommendations; SnapEDA_Link (none) -> https://www.snapeda.com/parts/PKLCS1212E4001-R1/Murata/view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
- R2: footprint Keebio-Parts:Resistor-Hybrid-Back -> _keebio-parts:Resistor-Hybrid-Back
- SW24, SW25, SW26, SW27, SW28, SW29, SW30, SW31, SW32, SW33, SW34, SW35, SW36, SW37, SW38, SW39, SW40, SW41, SW43, SW44, SW45, SW46, SW53, SW54, SW55, SW56, SW57, SW58: footprint Yoichiro:CherryMX_Choco_Hotswap -> _yoichiro:CherryMX_Choco_Hotswap; symbol kbd:SW_PUSH -> _kbd:SW_PUSH
- SW42: footprint kbd:ResetSW_1side -> _kbd:ResetSW; symbol kbd:SW_PUSH -> _kbd:SW_PUSH
- U2: footprint Yoichiro:Raspberry_Pi_Pico -> _yoichiro:Raspberry_Pi_Pico; symbol yoichiro:Raspberry_Pie_Pico -> _yoichiro:Raspberry_Pi_Pico
