File: pcb_tergo_mirrored/pcb_tergo_mirrored.kicad_sch (KiCad schematic)
At the start: 0 parts

Commit message: wip on PCB
Parts:
- added D1, D10, D11, D12, D13, D14, D15, D16, D17, D18, D19, D2, D20, D21, D22, D3, D4, D5, D50, D52, D58, D6, D60, D61, D62, D7, D8, D9: D, _keebio-parts:Diode-Hybrid-Back, symbol Device:D
- added J3: MJ-4PP-9, _kbd:MJ-4PP-9, symbol _kbd:MJ-4PP-9
- added JP?: Jumper_3_Open, Jumper:SolderJumper-3_P1.3mm_Open_Pad1.0x1.5mm, symbol Jumper:Jumper_3_Open
- added SW1, SW10, SW11, SW12, SW13, SW14, SW15, SW16, SW17, SW18, SW2, SW20, SW21, SW22, SW23, SW3, SW4, SW47, SW48, SW49, SW5, SW50, SW51, SW52, SW6, SW7, SW8, SW9: SW_PUSH, _yoichiro:CherryMX_Choco_Hotswap, symbol _kbd:SW_PUSH
- added SW19: SW_RESET, _kbd:ResetSW, symbol _kbd:SW_PUSH
- added U1: Raspberry_Pie_Pico, _prjlib:Raspberry_Pi_Pico_dual, symbol _prjlib:Raspberry_Pi_Pico
Connections:
- new net: D1.2 (A), SW1.2
- new net: D2.2 (A), SW2.2
- new net: D3.2 (A), SW3.2
- new net: D4.2 (A), SW4.2
- new net: D5.2 (A), SW5.2
- new net: D6.2 (A), SW6.2
- new net: D7.2 (A), SW7.2
- new net: D8.2 (A), SW8.2
- new net: D9.2 (A), SW9.2
- new net: D10.2 (A), SW10.2
- new net: D11.2 (A), SW11.2
- new net: D12.2 (A), SW12.2
- new net: D13.2 (A), SW13.2
- new net: D14.2 (A), SW14.2
- new net: D15.2 (A), SW15.2
- new net: D16.2 (A), SW16.2
- new net: D17.2 (A), SW17.2
- new net: D18.2 (A), SW18.2
- new net: D19.2 (A), SW20.2
- new net: D20.2 (A), SW21.2
- new net: D21.2 (A), SW22.2
- new net: D22.2 (A), SW23.2
- new net: JP?.2 (C), U1.29 (GP22)
- new net: D61.2 (A), SW52.2
- new net: D58.2 (A), SW49.2
- new net: D60.2 (A), SW51.2
- new net: D50.2 (A), SW47.2
- new net: D52.2 (A), SW48.2
- new net: D62.2 (A), SW50.2
- new net GND: J3.C, JP?.3 (B), SW19.2, U1.13 (GND), U1.18 (GND), U1.23 (GND), U1.28 (GND), U1.3 (GND), U1.38 (GND), U1.8 (GND)
- new net VCC: J3.D, JP?.1 (A), U1.39 (VSYS)
- new net audio-l: U1.11 (GP8)
- new net col0-l: SW1.1, SW10.1, SW2.1, SW3.1, SW47.1, U1.27 (GP21)
- new net col1-l: SW4.1, SW48.1, SW5.1, SW6.1, U1.26 (GP20)
- new net col2-l: SW49.1, SW7.1, SW8.1, SW9.1, U1.25 (GP19)
- new net col3-l: SW11.1, SW12.1, SW13.1, SW14.1, SW50.1, U1.24 (GP18)
- new net col4-l: SW15.1, SW16.1, SW17.1, SW18.1, SW51.1, U1.22 (GP17)
- new net col5-l: SW20.1, SW21.1, SW22.1, SW23.1, SW52.1, U1.21 (GP16)
- new net data-rx-l: J3.A, U1.2 (GP1)
- new net data-tx-l: J3.B, U1.1 (GP0)
- new net led-l: U1.9 (GP6)
- new net reset-l: SW19.1, U1.30 (RUN)
- new net row0-l: D50.1 (K), D52.1 (K), D58.1 (K), D60.1 (K), D61.1 (K), D62.1 (K), U1.15 (GP11)
- new net row1-l: D1.1 (K), D11.1 (K), D15.1 (K), D19.1 (K), D4.1 (K), D7.1 (K), U1.16 (GP12)
- new net row2-l: D12.1 (K), D16.1 (K), D2.1 (K), D20.1 (K), D5.1 (K), D8.1 (K), U1.17 (GP13)
- new net row3-l: D13.1 (K), D17.1 (K), D21.1 (K), D3.1 (K), D6.1 (K), D9.1 (K), U1.19 (GP14)
- new net row4-l: D10.1 (K), D14.1 (K), D18.1 (K), D22.1 (K), U1.20 (GP15)
- no-connect marks 0 -> 15
Other:
- removed sheet left part
- removed sheet right part
